Commit message: attempting to get gimballed camera on 1 axis

File: src/sjtu_drone_description/urdf/gen_xacro.urdf.xacro (robot description, xacro)
@@ -1,7 +1,9 @@
 <?xml version="1.0" ?>
-<robot name="sjtu_drone" xmlns:xacro="http://ros.org/wiki/xacro">
-  <xacro:arg name="drone_id" default="drone0"/>
-  <xacro:property name="drone_id" value="$(arg drone_id)"/>
-  <link name="${drone_id}/base_link">
+<!-- =================================================================================== -->
+<!-- |    This document was autogenerated by xacro from /workdir/src/sjtu_drone_description/urdf/sjtu_drone_multi.urdf.xacro | -->
+<!-- |    EDITING THIS FILE BY HAND IS NOT RECOMMENDED                                 | -->
+<!-- =================================================================================== -->
+<robot name="sjtu_drone">
+  <link name="drone1/base_link">
     <inertial>
       <mass value="1.477"/>
@@ -12,5 +14,5 @@
       <origin rpy="0 0 0" xyz="0   0   0.04"/>
       <geometry>
-        <mesh filename="file://$(find sjtu_drone_description)/models/sjtu_drone/quadrotor_4.stl"/>
+        <mesh filename="file:///workdir/install/sjtu_drone_description/share/sjtu_drone_description/models/sjtu_drone/quadrotor_4.stl"/>
         <!-- <mesh filename="package://sjtu_drone/quadrotor_4.stl"/> -->
       </geometry>
@@ -19,5 +21,5 @@
       <origin rpy="0 0 0" xyz="0   0   0.04"/>
       <geometry>
-        <mesh filename="file://$(find sjtu_drone_description)/models/sjtu_drone/quadrotor_4.dae"/>
+        <mesh filename="file:///workdir/install/sjtu_drone_description/share/sjtu_drone_description/models/sjtu_drone/quadrotor_4.dae"/>
         <!-- <mesh filename="package://sjtu_drone/quadrotor_4.dae"/> -->
       </geometry>
@@ -25,44 +27,44 @@
   </link>
   <!-- Front Camera Joint: Revolute on Y-axis -->
-<joint name="${drone_id}/front_cam_joint" type="revolute">
-  <origin rpy="0 0 0" xyz="0.2 0 0"/>
-  <parent link="${drone_id}/base_link"/>
-  <child link="${drone_id}/front_cam_link"/>
-  <axis xyz="0 1 0"/>
-  <limit effort="1.0" velocity="1.0" lower="-1.57" upper="1.57"/>
-  <dynamics damping="0.1" friction="0.1"/>
-  <ros2_control>
-    <hardware>
-      <plugin>fake_components/GenericSystem</plugin>
-    </hardware>
-    <command_interface name="position"/>
-    <state_interface name="position"/>
-    <state_interface name="velocity"/>
-  </ros2_control>
-</joint>
-<link name="${drone_id}/front_cam_link">
-  <visual>
-    <geometry>
-      <cylinder length="0.1" radius="0.01"/>
-    </geometry>
-    <material name="Blue">
-      <color rgba="0.0 0.0 1.0 1.0"/>
-    </material>
-  </visual>
-  <collision>
-    <geometry>
-      <cylinder length="0.1" radius="0.01"/>
-    </geometry>
-  </collision>
-  <inertial>
-    <mass value="0.1"/>
-    <inertia ixx="0.0001" ixy="0" ixz="0" iyy="0.0001" iyz="0" izz="0.0002"/>
-  </inertial>
-</link>
+  <joint name="drone1/front_cam_joint" type="revolute">
+    <origin rpy="0 0 0" xyz="0.2 0 0"/>
+    <parent link="drone1/base_link"/>
+    <child link="drone1/front_cam_link"/>
+    <axis xyz="0 1 0"/>
+    <limit effort="1.0" lower="-1.57" upper="1.57" velocity="1.0"/>
+    <dynamics damping="0.1" friction="0.1"/>
+    <ros2_control>
+      <hardware>
+        <plugin>fake_components/GenericSystem</plugin>
+      </hardware>
+      <command_interface name="position"/>
+      <state_interface name="position"/>
+      <state_interface name="velocity"/>
+    </ros2_control>
+  </joint>
+  <link name="drone1/front_cam_link">
+    <visual>
+      <geometry>
+        <cylinder length="0.1" radius="0.01"/>
+      </geometry>
+      <material name="Blue">
+        <color rgba="0.0 0.0 1.0 1.0"/>
+      </material>
+    </visual>
+    <collision>
+      <geometry>
+        <cylinder length="0.1" radius="0.01"/>
+      </geometry>
+    </collision>
+    <inertial>
+      <mass value="0.1"/>
+      <inertia ixx="0.0001" ixy="0" ixz="0" iyy="0.0001" iyz="0" izz="0.0002"/>
+    </inertial>
+  </link>
   <gazebo>
-    <plugin name='simple_drone' filename='libplugin_drone.so'>
-      <bodyName>${drone_id}/base_link</bodyName>
-      <rosNamespace>${drone_id}</rosNamespace>
-      <imuTopic>${drone_id}/imu</imuTopic>
+    <plugin filename="libplugin_drone.so" name="simple_drone">
+      <bodyName>drone1/base_link</bodyName>
+      <rosNamespace>drone1</rosNamespace>
+      <imuTopic>drone1/imu</imuTopic>
       <rollpitchProportionalGain>10.0</rollpitchProportionalGain>
       <rollpitchDifferentialGain>5.0</rollpitchDifferentialGain>
@@ -93,17 +95,17 @@
   </gazebo>
   <gazebo>
-    <plugin name="gazebo_ros_joint_state_publisher" filename="libgazebo_ros_joint_state_publisher.so">
-      <joint_name>${drone_id}/front_cam_joint</joint_name>
+    <plugin filename="libgazebo_ros_joint_state_publisher.so" name="gazebo_ros_joint_state_publisher">
+      <joint_name>drone1/front_cam_joint</joint_name>
     </plugin>
   </gazebo>
   <!-- Sensors -->
   <!-- IMU sensor in 100fps -->
-  <gazebo reference="${drone_id}/base_link">
-    <sensor name='sensor_imu' type='imu'>
+  <gazebo reference="drone1/base_link">
+    <sensor name="sensor_imu" type="imu">
       <always_on> 1 </always_on>
       <visualize>1</visualize>
       <update_rate> 100 </update_rate>
       <pose> 0 0 0 0 0 0 </pose>
-      <plugin name='imu' filename='libgazebo_ros_imu_sensor.so'>
+      <plugin filename="libgazebo_ros_imu_sensor.so" name="imu">
         <initial_orientation_as_reference>false</initial_orientation_as_reference>
       </plugin>
@@ -124,5 +126,5 @@
   </gazebo>
   <!-- Front Camera Sensor -->
- <gazebo reference="${drone_id}/front_cam_link">
+  <gazebo reference="drone1/front_cam_link">
     <sensor name="front_camera" type="camera">
       <camera>
@@ -146,5 +148,5 @@
       <update_rate>60</update_rate>
       <visualize>true</visualize>
-      <plugin name="camera_front" filename="libgazebo_ros_camera.so">
+      <plugin filename="libgazebo_ros_camera.so" name="camera_front">
         <ros>
           <remapping>image_raw:=camera_front</remapping>
