Commit message: work on one camera

File: src/sjtu_drone_description/urdf/sjtu_drone_multi.urdf.xacro (robot description, xacro)
@@ -25,15 +25,9 @@
   </link>
   <joint name="${drone_id}/front_cam_joint" type="fixed">
-    <origin rpy="0 0.261799 0" xyz="0.2 0 0"/>
+    <origin rpy="0 0 0" xyz="0.2 0 0"/>
     <parent link="${drone_id}/base_link" />
     <child link="${drone_id}/front_cam_link" />
   </joint>
   <link name="${drone_id}/front_cam_link"/>
-  <joint name="${drone_id}/bottom_cam_joint" type="fixed">
-    <origin rpy="0 1.570796326794897 0" xyz="0 0 0"/>
-    <parent link="${drone_id}/base_link" />
-    <child link="${drone_id}/bottom_cam_link" />
-  </joint>
-  <link name="${drone_id}/bottom_cam_link"/>
   <gazebo>
     <plugin name='simple_drone' filename='libplugin_drone.so'>
@@ -127,37 +121,3 @@
     </sensor>
   </gazebo>
-  <!-- downward looking camera -->
-  <gazebo reference="${drone_id}/bottom_cam_link">
-    <sensor name="down_camera" type="camera">
-      <camera>
-        <horizontal_fov>1.047</horizontal_fov>
-        <image>
-          <width>640</width>
-          <height>360</height>
-          <format>R8G8B8</format>
-        </image>
-        <clip>
-          <near>0.1</near>
-          <far>100</far>
-        </clip>
-        <noise>
-          <type>gaussian</type>
-          <mean>0.0</mean>
-          <stddev>0.005</stddev>
-        </noise>
-      </camera>
-      <always_on>1</always_on>
-      <update_rate>15</update_rate>
-      <visualize>true</visualize>
-      <plugin name="camera_bottom" filename="libgazebo_ros_camera.so">
-        <ros>
-          <remapping>image_raw:=camera_bottom</remapping>
-          <remapping>camera_info:=camera_bottom_info</remapping>
-        </ros>
-        <camera_name>bottom</camera_name>
-        <frame_name>bottom_cam_link</frame_name>
-        <hack_baseline>0.07</hack_baseline>
-      </plugin>
-    </sensor>
-  </gazebo>
 </robot>

Commit message: revert and add ros2 control to dockerfile

File: src/sjtu_drone_description/urdf/sjtu_drone_multi.urdf.xacro (robot description, xacro)
@@ -24,12 +24,11 @@
     </visual>
   </link>
-  <!-- Front Camera Joint: Revolute on Y-axis -->
 <joint name="${drone_id}/front_cam_joint" type="revolute">
-  <origin rpy="0 0 0" xyz="0.2 0 0"/>
+  <origin rpy="0 0 0" xyz="0.2 0 0.05"/>
   <parent link="${drone_id}/base_link"/>
   <child link="${drone_id}/front_cam_link"/>
   <axis xyz="0 1 0"/>
   <limit effort="1.0" velocity="1.0" lower="-1.57" upper="1.57"/>
-  <dynamics damping="0.1" friction="0.1"/>
+  <dynamics damping="0.0" friction="0.0"/>
   <ros2_control>
     <hardware>
@@ -44,5 +43,5 @@
   <visual>
     <geometry>
-      <cylinder length="0.1" radius="0.01"/>
+      <cylinder length="0.05" radius="0.025"/>
     </geometry>
     <material name="Blue">
@@ -52,10 +51,10 @@
   <collision>
     <geometry>
-      <cylinder length="0.1" radius="0.01"/>
+      <cylinder length="0.025" radius="0.025"/>
     </geometry>
   </collision>
   <inertial>
-    <mass value="0.1"/>
-    <inertia ixx="0.0001" ixy="0" ixz="0" iyy="0.0001" iyz="0" izz="0.0002"/>
+    <mass value="0.01"/>
+    <inertia ixx="0.001" ixy="0" ixz="0" iyy="0.001" iyz="0" izz="0.002"/>
   </inertial>
 </link>
@@ -86,13 +85,8 @@
       <positionZIntegralGain>0.0</positionZIntegralGain>
       <positionZLimit>-1</positionZLimit>
-      <maxForce>300</maxForce>
+      <maxForce>10000</maxForce>
       <motionSmallNoise>0.05</motionSmallNoise>
       <motionDriftNoise>0.03</motionDriftNoise>
       <motionDriftNoiseTime>5.0</motionDriftNoiseTime>
-    </plugin>
-  </gazebo>
-  <gazebo>
-    <plugin name="gazebo_ros_joint_state_publisher" filename="libgazebo_ros_joint_state_publisher.so">
-      <joint_name>${drone_id}/front_cam_joint</joint_name>
     </plugin>
   </gazebo>
@@ -123,5 +117,4 @@
     </sensor>
   </gazebo>
-  <!-- Front Camera Sensor -->
  <gazebo reference="${drone_id}/front_cam_link">
     <sensor name="front_camera" type="camera">
