Commit message: camera adjusted

File: src/sjtu_drone_description/urdf/robot_core_lr.xacro (robot description, xacro)
@@ -1,165 +1,90 @@
 <?xml version="1.0"?>
 <robot xmlns:xacro="http://www.ros.org/wiki/xacro">
-	<xacro:include filename="inertial_macros.xacro"/>
-	<gazebo reference="${drone_id}/base_link">
-		<static>true</static>
-	</gazebo>
-	<!-- STAND_LINK -->
-	<joint name="stand_joint" type="fixed">
-		<parent link="${drone_id}/base_link"/>
-		<child link="stand_link"/>
-		<origin xyz="0 0 0"/>
-	</joint>
-	<link name="stand_link">
-		<visual>
-			<origin xyz="0 0 0.2"/>
-			<geometry>
-				<cylinder radius="0.05" length="0.1"/>
-			</geometry>
-		</visual>
-		<collision>
-			<origin xyz="0 0 0.2"/>
-			<geometry>
-				<cylinder radius="0.05" length="0.1"/>
-			</geometry>
-		</collision>
-		<xacro:inertial_cylinder mass="0.05" length="0.4" radius="0.5">
-            <origin xyz="0 0 0.2" rpy="0 0 0"/>
-        </xacro:inertial_cylinder>
-	</link>
-	<gazebo reference="stand_link">
-		<material>Gazebo/Red</material>
-		<mu1 value="10"/>
-		<mu2 value="10"/>
-	</gazebo>
-	<!-- AX1_LINK -->
-	<joint name="ax1_joint" type="revolute">
-		<parent link="stand_link"/>
-		<child link="ax1_link"/>
-		<limit effort="10" velocity="1" upper="${pi*2}" lower="${-pi*2}"/>
-		<axis xyz="0 0 1"/>
-		<origin xyz="0 0 0.2"/>
-		<dynamics damping="10.0" friction="10.0"/>
-	</joint>
-	<link name="ax1_link">
-		<visual>
-			<origin xyz="0 0 0.01"/>
-			<geometry>
-				<box size="0.1 0.1 0.1"/>
-			</geometry>
-		</visual>
-		<collision>
-			<origin xyz="0 0 0"/>
-			<geometry>
-				<box size="0.1 0.1 0.1"/>
-			</geometry>
-		</collision>
-		<xacro:inertial_box mass="0.05" x="0.1" y="0.1" z="0.1">
+    <xacro:include filename="inertial_macros.xacro"/>
+    <!-- AX1_LINK -->
+    <joint name="ax1_joint" type="revolute">
+        <parent link="${drone_id}/base_link"/>
+        <child link="ax1_link"/>
+        <limit effort="10" velocity="1" upper="${pi*2}" lower="${-pi*2}"/>
+        <axis xyz="0 0 1"/>
+        <origin xyz="0 0 0.2"/>
+        <dynamics damping="10.0" friction="10.0"/>
+    </joint>
+    <link name="ax1_link">
+        <xacro:inertial_box mass="0.05" x="0.1" y="0.1" z="0.1">
             <origin xyz="0 0 0.2" rpy="0 0 0"/>
         </xacro:inertial_box>
-	</link>
-	<gazebo reference="ax1_link">
-		<material>Gazebo/Red</material>
-		<mu1 value="10"/>
-		<mu2 value="10"/>
-	</gazebo>
-	<!-- AX2_LINK -->
-	<joint name="ax2_joint" type="revolute">
-		<parent link="ax1_link"/>
-		<child link="ax2_link"/>
-		<limit effort="10" velocity="1" upper="${pi/2}" lower="${-pi/2}"/>
-		<origin xyz="0 0 0.2"/>
-		<axis xyz="1 0 0"/>
-		<dynamics damping="10.0" friction="10.0"/>
-	</joint>
-	<link name="ax2_link">
-		<visual>
-			<origin xyz="0 0 0"/>
-			<geometry>
-				<box size="0.1 0.1 0.1"/>
-			</geometry>
-		</visual>
-		<collision>
-			<origin xyz="0 0 0.01"/>
-			<geometry>
-				<box size="0.1 0.1 0.1"/>
-			</geometry>
-		</collision>
-		<xacro:inertial_box mass="0.05" x="0.1" y="0.1" z="0.1">
+    </link>
+    <gazebo reference="ax1_link">
+        <material>Gazebo/Red</material>
+        <mu1 value="10"/>
+        <mu2 value="10"/>
+    </gazebo>
+    <!-- AX2_LINK -->
+    <joint name="ax2_joint" type="revolute">
+        <parent link="ax1_link"/>
+        <child link="ax2_link"/>
+        <limit effort="10" velocity="1" upper="${pi/2}" lower="${-pi/2}"/>
+        <origin xyz="0 0 0.2"/>
+        <axis xyz="1 0 0"/>
+        <dynamics damping="10.0" friction="10.0"/>
+    </joint>
+    <link name="ax2_link">
+        <xacro:inertial_box mass="0.05" x="0.1" y="0.1" z="0.1">
             <origin xyz="0 0 0.2" rpy="0 0 0"/>
         </xacro:inertial_box>
-	</link>
-	<gazebo reference="ax2_link">
-		<material>Gazebo/Black</material>
-		<mu1 value="10"/>
-		<mu2 value="10"/>
-	</gazebo>
-<!-- camera link -->
-  <joint name="camera_link" type="fixed">
-    <origin rpy="0 ${-pi/2} 0" xyz="0 0 0"/>
-    <parent link="ax2_link" />
-    <child link="camera_link" />
-  </joint>
-  <link name="camera_link"/>
-<!-- controller -->
-	<ros2_control name="GazeboSystem" type="system">
-    	<hardware>
-      		<plugin>gazebo_ros2_control/GazeboSystem</plugin>
-    	</hardware>
-		<joint name="ax1_joint">
-      		<command_interface name="position">
-        		<param name="min">${-pi*2}</param>
-        		<param name="max">${pi*2}</param>
-      		</command_interface>
-      		<state_interface name="position">
-				<param name="initial_value">${0}</param>
-			</state_interface>
-      		<state_interface name="velocity"/>
-      		<!--<state_interface name="effort"/>-->
-    	</joint>
-    	<joint name="ax2_joint">
-      		<command_interface name="position">
-        		<param name="min">${-pi/2}</param>
-        		<param name="max">${pi/2}</param>
-      		</command_interface>
-      		<state_interface name="position">
-				<param name="initial_value">${0}</param>
-			</state_interface>
-      		<state_interface name="velocity"/>
-      		<!--<state_interface name="effort"/>-->
-    	</joint>
-  	</ros2_control>
- <gazebo reference="camera_link">
-    <sensor name="front_camera" type="camera">
-      <camera>
-        <horizontal_fov>2.09</horizontal_fov>
-        <image>
-          <width>960</width>
-          <height>540</height>
-          <format>R8G8B8</format>
-        </image>
-        <clip>
-          <near>0.1</near>
-          <far>100</far>
-        </clip>
-        <noise>
-          <type>gaussian</type>
-          <mean>0.0</mean>
-          <stddev>0.005</stddev>
-        </noise>
-      </camera>
-      <always_on>1</always_on>
-      <update_rate>60</update_rate>
-      <visualize>true</visualize>
-      <plugin name="camera_front" filename="libgazebo_ros_camera.so">
-        <ros>
-          <remapping>image_raw:=camera_front</remapping>
-          <remapping>camera_info:=camera_front_info</remapping>
-        </ros>
-        <camera_name>front</camera_name>
-        <frame_name>front_cam_link</frame_name>
-        <hack_baseline>0.07</hack_baseline>
-      </plugin>
-    </sensor>
-  </gazebo>
+    </link>
+    <gazebo reference="ax2_link">
+        <material>Gazebo/Black</material>
+        <mu1 value="10"/>
+        <mu2 value="10"/>
+    </gazebo>
+    <!-- Camera Link -->
+    <joint name="camera_joint" type="fixed">
+        <origin rpy="0 0 0" xyz="0.2 0 0.075"/>
+        <parent link="${drone_id}/base_link"/>
+        <child link="camera_link"/>
+    </joint>
+    <link name="camera_link">
+        <visual>
+            <origin xyz="0 0 0" rpy="0 0 0"/>
+            <geometry>
+                <box size="0.025 0.025 0.025"/>
+            </geometry>
+        </visual>
+    </link>
+    <!-- Camera Sensor -->
+    <gazebo reference="camera_link">
+        <sensor name="front_camera" type="camera">
+            <camera>
+                <horizontal_fov>2.09</horizontal_fov>
+                <image>
+                    <width>960</width>
+                    <height>540</height>
+                    <format>R8G8B8</format>
+                </image>
+                <clip>
+                    <near>0.1</near>
+                    <far>100</far>
+                </clip>
+                <noise>
+                    <type>gaussian</type>
+                    <mean>0.0</mean>
+                    <stddev>0.005</stddev>
+                </noise>
+            </camera>
+            <always_on>1</always_on>
+            <update_rate>60</update_rate>
+            <visualize>true</visualize>
+            <plugin name="camera_front" filename="libgazebo_ros_camera.so">
+                <ros>
+                    <remapping>image_raw:=camera_front</remapping>
+                    <remapping>camera_info:=camera_front_info</remapping>
+                </ros>
+                <camera_name>front</camera_name>
+                <frame_name>front_cam_link</frame_name>
+                <hack_baseline>0.07</hack_baseline>
+            </plugin>
+        </sensor>
+    </gazebo>
 </robot>

Commit message: update

File: src/sjtu_drone_description/urdf/robot_core_lr.xacro (robot description, xacro)
@@ -54,4 +54,32 @@
         </visual>
     </link>
+<!-- controller -->
+	<ros2_control name="GazeboSystem" type="system">
+    	<hardware>
+      		<plugin>gazebo_ros2_control/GazeboSystem</plugin>
+    	</hardware>
+		<joint name="ax1_joint">
+      		<command_interface name="position">
+        		<param name="min">${-pi*2}</param>
+        		<param name="max">${pi*2}</param>
+      		</command_interface>
+      		<state_interface name="position">
+				<param name="initial_value">${0}</param>
+			</state_interface>
+      		<state_interface name="velocity"/>
+      		<!--<state_interface name="effort"/>-->
+    	</joint>
+    	<joint name="ax2_joint">
+      		<command_interface name="position">
+        		<param name="min">${-pi/2}</param>
+        		<param name="max">${pi/2}</param>
+      		</command_interface>
+      		<state_interface name="position">
+				<param name="initial_value">${0}</param>
+			</state_interface>
+      		<state_interface name="velocity"/>
+      		<!--<state_interface name="effort"/>-->
+    	</joint>
+  	</ros2_control>
     <!-- Camera Sensor -->
     <gazebo reference="camera_link">

Commit message: try only to spawn camera

File: src/sjtu_drone_description/urdf/robot_core_lr.xacro (robot description, xacro)
@@ -2,7 +2,13 @@
 <robot xmlns:xacro="http://www.ros.org/wiki/xacro">
     <xacro:include filename="inertial_macros.xacro"/>
+	<link name="world">
+		<origin xyz="0 0 0.0"/>
+	</link>
+	<gazebo reference="world">
+		<static>true</static>
+	</gazebo>
     <!-- AX1_LINK -->
     <joint name="${drone_id}/ax1_joint" type="revolute">
-        <parent link="${drone_id}/base_link"/>
+        <parent link="world"/>
         <child link="${drone_id}/ax1_link"/>
         <limit effort="10" velocity="1" upper="${pi*2}" lower="${-pi*2}"/>
@@ -43,5 +49,5 @@
     <joint name="${drone_id}/camera_joint" type="fixed">
         <origin rpy="0 0 0" xyz="0.2 0 0.075"/>
-        <parent link="${drone_id}/base_link"/>
+        <parent link="${drone_id}/ax2_link"/>
         <child link="${drone_id}/camera_link"/>
     </joint>

File: src/sjtu_drone_description/urdf/sjtu_drone_multi.urdf.xacro (robot description, xacro)
@@ -3,34 +3,5 @@
   <xacro:arg name="drone_id" default="drone0"/>
   <xacro:property name="drone_id" value="$(arg drone_id)"/>
-  <link name="${drone_id}/robot_root"/>
-  <!-- Fixed joint from dummy root to the actual base_link -->
-  <joint name="${drone_id}/root_joint" type="fixed">
-    <parent link="${drone_id}/robot_root"/>
-    <child link="${drone_id}/base_link"/>
-    <!-- No offset, or if you want to shift the base, do so here -->
-    <origin xyz="0 0 0" rpy="0 0 0"/>
-  </joint>
-  <link name="${drone_id}/base_link">
-    <inertial>
-      <mass value="1.477"/>
-      <origin rpy="0 0 0" xyz="0 0 0"/>
-      <inertia ixx="0.1152" ixy="0" ixz="0" iyy="0.1152" iyz="0" izz="0.218"/>
-    </inertial>
-    <collision name="sjtu_drone_collision">
-      <origin rpy="0 0 0" xyz="0   0   0.04"/>
-      <geometry>
-        <mesh filename="file://$(find sjtu_drone_description)/models/sjtu_drone/quadrotor_4.stl"/>
-        <!-- <mesh filename="package://sjtu_drone/quadrotor_4.stl"/> -->
-      </geometry>
-    </collision>
-    <visual name="sjtu_drone_visual">
-      <origin rpy="0 0 0" xyz="0   0   0.04"/>
-      <geometry>
-        <mesh filename="file://$(find sjtu_drone_description)/models/sjtu_drone/quadrotor_4.dae"/>
-        <!-- <mesh filename="package://sjtu_drone/quadrotor_4.dae"/> -->
-      </geometry>
-    </visual>
-  </link>
-  <gazebo>
+  <!-- <gazebo>
     <plugin name='simple_drone' filename='libplugin_drone.so'>
       <bodyName>${drone_id}/base_link</bodyName>
@@ -63,8 +34,8 @@
       <motionDriftNoiseTime>5.0</motionDriftNoiseTime>
     </plugin>
-  </gazebo>
+  </gazebo> -->
   <!-- Sensors -->
   <!-- IMU sensor in 100fps -->
-  <gazebo reference="${drone_id}/base_link">
+  <!-- <gazebo reference="${drone_id}/base_link">
     <sensor name='sensor_imu' type='imu'>
       <always_on> 1 </always_on>
@@ -89,5 +60,5 @@
       </imu>
     </sensor>
-  </gazebo>
+  </gazebo> -->
   	<xacro:include filename="robot_core_lr.xacro"/>
     <xacro:include filename="gazebo_control.xacro"/>
