Commit message: added standalone gimbal

File: src/sjtu_drone_description/urdf/gimbal_camera_description.xacro (robot description, xacro)
@@ -1,23 +1,17 @@
 <?xml version="1.0"?>
 <robot xmlns:xacro="http://www.ros.org/wiki/xacro">
-    <xacro:include filename="inertial_macros.xacro"/>
-	<link name="world">
-		<origin xyz="0 0 0.0"/>
-	</link>
-	<gazebo reference="world">
-		<static>true</static>
-	</gazebo>
+    <xacro:include filename="gimbal_camera_inertial_macros.xacro"/>
     <!-- AX1_LINK -->
     <joint name="${drone_id}/ax1_joint" type="revolute">
-        <parent link="world"/>
+        <parent link="${drone_id}/base_link"/>
         <child link="${drone_id}/ax1_link"/>
         <limit effort="10" velocity="1" upper="${pi*2}" lower="${-pi*2}"/>
         <axis xyz="0 0 1"/>
-        <origin xyz="0 0 0.2"/>
+        <origin xyz="0 0 0.1"/>
         <dynamics damping="10.0" friction="10.0"/>
     </joint>
     <link name="${drone_id}/ax1_link">
         <xacro:inertial_box mass="0.05" x="0.1" y="0.1" z="0.1">
-            <origin xyz="0 0 0.2" rpy="0 0 0"/>
+            <origin xyz="0 0 0.1" rpy="0 0 0"/>
         </xacro:inertial_box>
     </link>
@@ -32,5 +26,5 @@
         <child link="${drone_id}/ax2_link"/>
         <limit effort="10" velocity="1" upper="${pi/2}" lower="${-pi/2}"/>
-        <origin xyz="0 0 0.2"/>
+        <origin xyz="0 0 0.1"/>
         <axis xyz="1 0 0"/>
         <dynamics damping="10.0" friction="10.0"/>
@@ -38,5 +32,5 @@
     <link name="${drone_id}/ax2_link">
         <xacro:inertial_box mass="0.05" x="0.1" y="0.1" z="0.1">
-            <origin xyz="0 0 0.2" rpy="0 0 0"/>
+            <origin xyz="0 0 0.1" rpy="0 0 0"/>
         </xacro:inertial_box>
     </link>
@@ -71,5 +65,5 @@
       		</command_interface>
       		<state_interface name="position">
-				<param name="initial_value">${pi/4}</param>
+				<param name="initial_value">${pi/12}</param>
 			</state_interface>
       		<state_interface name="velocity"/>
@@ -82,5 +76,5 @@
       		</command_interface>
       		<state_interface name="position">
-				<param name="initial_value">${pi/4}</param>
+				<param name="initial_value">${pi/12}</param>
 			</state_interface>
       		<state_interface name="velocity"/>

File: src/sjtu_drone_description/urdf/sjtu_drone_base.xacro (robot description, xacro)
@@ -1,6 +1,4 @@
 <?xml version="1.0" ?>
 <robot name="sjtu_drone" xmlns:xacro="http://ros.org/wiki/xacro">
-  <xacro:arg name="drone_id" default="drone0"/>
-  <xacro:property name="drone_id" value="$(arg drone_id)"/>
   <link name="${drone_id}/base_link">
     <inertial>
