Commit message: more testing

File: src/sjtu_drone_description/urdf_no_ns/gimbal_camera_description.xacro (robot description, xacro)
@@ -6,5 +6,5 @@
         <parent link="base_link"/>
         <child link="ax1_link"/>
-        <limit effort="10" velocity="1" upper="${pi*2}" lower="${-pi*2}"/>
+        <limit effort="1.0" velocity="1" upper="${pi*2}" lower="${-pi*2}"/>
         <axis xyz="0 0 1"/>
         <origin xyz="0 0 0.1"/>
@@ -25,5 +25,5 @@
         <parent link="ax1_link"/>
         <child link="ax2_link"/>
-        <limit effort="10" velocity="1" upper="${pi/2}" lower="${-pi/2}"/>
+        <limit effort="1.0" velocity="1" upper="${pi/2}" lower="${-pi/2}"/>
         <origin xyz="0 0 0.1"/>
         <axis xyz="1 0 0"/>

Commit message: works with no namespace

File: src/sjtu_drone_description/urdf_no_ns/gimbal_camera_description.xacro (robot description, xacro)
@@ -7,11 +7,11 @@
         <child link="ax1_link"/>
         <limit effort="1.0" velocity="1" upper="${pi*2}" lower="${-pi*2}"/>
-        <axis xyz="0 0 1"/>
-        <origin xyz="0 0 0.1"/>
+        <axis xyz="1 0 0"/>
+        <origin xyz="0.3 0 0.075"/>
         <dynamics damping="0.1" friction="0.1"/>
     </joint>
     <link name="ax1_link">
         <xacro:inertial_box mass="0.01" x="0.1" y="0.1" z="0.1">
-            <origin xyz="0 0 0.1" rpy="0 0 0"/>
+            <origin xyz="0.3 0 0.075" rpy="0 0 0"/>
         </xacro:inertial_box>
     </link>
@@ -26,11 +26,11 @@
         <child link="ax2_link"/>
         <limit effort="1.0" velocity="1" upper="${pi/2}" lower="${-pi/2}"/>
-        <origin xyz="0 0 0.1"/>
-        <axis xyz="1 0 0"/>
+        <origin xyz="0 0 0"/>
+        <axis xyz="0 1 0"/>
         <dynamics damping="0.1" friction="0.1"/>
     </joint>
     <link name="ax2_link">
         <xacro:inertial_box mass="0.01" x="0.1" y="0.1" z="0.1">
-            <origin xyz="0 0 0.1" rpy="0 0 0"/>
+            <origin xyz="0 0 0" rpy="0 0 0"/>
         </xacro:inertial_box>
     </link>
@@ -42,5 +42,5 @@
     <!-- Camera Link -->
     <joint name="camera_joint" type="fixed">
-        <origin rpy="0 0 0" xyz="0.2 0 0.075"/>
+        <origin rpy="0 0 0" xyz="0 0 0"/>
         <parent link="ax2_link"/>
         <child link="camera_link"/>
@@ -88,6 +88,6 @@
                 <horizontal_fov>2.09</horizontal_fov>
                 <image>
-                    <width>960</width>
-                    <height>540</height>
+                    <width>800</width>
+                    <height>800</height>
                     <format>R8G8B8</format>
                 </image>

Commit message: update

File: src/sjtu_drone_description/urdf_no_ns/gimbal_camera_description.xacro (robot description, xacro)
@@ -12,6 +12,6 @@
     </joint>
     <link name="ax1_link">
-        <xacro:inertial_box mass="0.01" x="0.1" y="0.1" z="0.1">
-            <origin xyz="0.3 0 0.075" rpy="0 0 0"/>
+        <xacro:inertial_box mass="0.001" x="0.025" y="0.025" z="0.025">
+            <origin xyz="0 0 0" rpy="0 0 0"/>
         </xacro:inertial_box>
     </link>
@@ -31,5 +31,5 @@
     </joint>
     <link name="ax2_link">
-        <xacro:inertial_box mass="0.01" x="0.1" y="0.1" z="0.1">
+        <xacro:inertial_box mass="0.001" x="0.025" y="0.025" z="0.025">
             <origin xyz="0 0 0" rpy="0 0 0"/>
         </xacro:inertial_box>

File: src/sjtu_drone_description/urdf_no_ns/sjtu_drone_base.xacro (robot description, xacro)
@@ -3,5 +3,5 @@
   <link name="base_link">
     <inertial>
-      <mass value="14.77"/>
+      <mass value="1.477"/>
       <origin rpy="0 0 0" xyz="0 0 0"/>
       <inertia ixx="0.1152" ixy="0" ixz="0" iyy="0.1152" iyz="0" izz="0.218"/>

Commit message: progress on camera tracking

File: src/sjtu_drone_description/urdf_no_ns/gimbal_camera_description.xacro (robot description, xacro)
@@ -6,8 +6,8 @@
         <parent link="base_link"/>
         <child link="ax1_link"/>
-        <limit effort="1.0" velocity="1" upper="${pi*2}" lower="${-pi*2}"/>
+        <limit effort="0.1" velocity="1" upper="${pi*2}" lower="${-pi*2}"/>
         <axis xyz="1 0 0"/>
         <origin xyz="0.3 0 0.075"/>
-        <dynamics damping="0.1" friction="0.1"/>
+        <dynamics damping="0.001" friction="0.001"/>
     </joint>
     <link name="ax1_link">
@@ -25,8 +25,8 @@
         <parent link="ax1_link"/>
         <child link="ax2_link"/>
-        <limit effort="1.0" velocity="1" upper="${pi/2}" lower="${-pi/2}"/>
+        <limit effort="0.1" velocity="1" upper="${pi/2}" lower="${-pi/2}"/>
         <origin xyz="0 0 0"/>
         <axis xyz="0 1 0"/>
-        <dynamics damping="0.1" friction="0.1"/>
+        <dynamics damping="0.001" friction="0.001"/>
     </joint>
     <link name="ax2_link">
