Commit message: simplified to turretted camera, need to work on cv tracking

File: src/sjtu_drone_description/urdf_turret/gimbal_camera_description.xacro (robot description, xacro)
@@ -6,6 +6,6 @@
         <parent link="base_link"/>
         <child link="ax1_link"/>
-        <limit effort="0.1" velocity="1" upper="${pi*2}" lower="${-pi*2}"/>
-        <axis xyz="1 0 0"/>
+        <limit effort="0.1" velocity="1" upper="${pi/3}" lower="${-pi/3}"/>
+        <axis xyz="0 0 1"/>
         <origin xyz="0.3 0 0.075"/>
         <dynamics damping="0.001" friction="0.001"/>
@@ -25,5 +25,5 @@
         <parent link="ax1_link"/>
         <child link="ax2_link"/>
-        <limit effort="0.1" velocity="1" upper="${pi/2}" lower="${-pi/2}"/>
+        <limit effort="0.1" velocity="1" upper="${pi/3}" lower="${-pi/3}"/>
         <origin xyz="0 0 0"/>
         <axis xyz="0 1 0"/>
