Commit message: update for testing with dockerfile

File: src/sjtu_drone_description/urdf_multi/sjtu_drone_multi.xacro (robot description, xacro)
@@ -1,5 +1,7 @@
 <?xml version="1.0" ?>
 <robot name="sjtu_drone" xmlns:xacro="http://ros.org/wiki/xacro">
-  <link name="base_link">
+  <xacro:arg name="drone_id" default="drone0"/>
+  <xacro:property name="drone_id" value="$(arg drone_id)"/>
+  <link name="${drone_id}/base_link">
     <inertial>
       <mass value="1.477"/>
@@ -22,8 +24,21 @@
     </visual>
   </link>
+  <joint name="${drone_id}/front_cam_joint" type="fixed">
+    <origin rpy="0 0.261799 0" xyz="0.2 0 0"/>
+    <parent link="${drone_id}/base_link" />
+    <child link="${drone_id}/front_cam_link" />
+  </joint>
+  <link name="${drone_id}/front_cam_link"/>
+  <joint name="${drone_id}/bottom_cam_joint" type="fixed">
+    <origin rpy="0 1.570796326794897 0" xyz="0 0 0"/>
+    <parent link="${drone_id}/base_link" />
+    <child link="${drone_id}/bottom_cam_link" />
+  </joint>
+  <link name="${drone_id}/bottom_cam_link"/>
   <gazebo>
     <plugin name='simple_drone' filename='libplugin_drone.so'>
-      <bodyName>base_link</bodyName>
-      <imuTopic>imu</imuTopic>
+      <bodyName>${drone_id}/base_link</bodyName>
+      <rosNamespace>${drone_id}</rosNamespace>
+      <imuTopic>${drone_id}/imu</imuTopic>
       <rollpitchProportionalGain>10.0</rollpitchProportionalGain>
       <rollpitchDifferentialGain>5.0</rollpitchDifferentialGain>
@@ -47,5 +62,5 @@
       <positionZIntegralGain>0.0</positionZIntegralGain>
       <positionZLimit>-1</positionZLimit>
-      <maxForce>10000</maxForce>
+      <maxForce>300</maxForce>
       <motionSmallNoise>0.05</motionSmallNoise>
       <motionDriftNoise>0.03</motionDriftNoise>
@@ -55,5 +70,5 @@
   <!-- Sensors -->
   <!-- IMU sensor in 100fps -->
-  <gazebo reference="base_link">
+  <gazebo reference="${drone_id}/base_link">
     <sensor name='sensor_imu' type='imu'>
       <always_on> 1 </always_on>
@@ -79,3 +94,36 @@
     </sensor>
   </gazebo>
+ <gazebo reference="${drone_id}/front_cam_link">
+    <sensor name="front_camera" type="camera">
+      <camera>
+        <horizontal_fov>2.09</horizontal_fov>
+        <image>
+          <width>960</width>
+          <height>540</height>
+          <format>R8G8B8</format>
+        </image>
+        <clip>
+          <near>0.1</near>
+          <far>100</far>
+        </clip>
+        <noise>
+          <type>gaussian</type>
+          <mean>0.0</mean>
+          <stddev>0.005</stddev>
+        </noise>
+      </camera>
+      <always_on>1</always_on>
+      <update_rate>60</update_rate>
+      <visualize>true</visualize>
+      <plugin name="camera_front" filename="libgazebo_ros_camera.so">
+        <ros>
+          <remapping>image_raw:=camera_front</remapping>
+          <remapping>camera_info:=camera_front_info</remapping>
+        </ros>
+        <camera_name>front</camera_name>
+        <frame_name>front_cam_link</frame_name>
+        <hack_baseline>0.07</hack_baseline>
+      </plugin>
+    </sensor>
+  </gazebo>
 </robot>
